Commit message: keyboard teleop

File: ros_ws/src/motor_p/urdf/motor.urdf (robot description, URDF)
Before this commit: robot motor_urdf, 2 links, 1 joints
Links:
- removed link right_leg
- added link propeller; visual box size=0.05 0.02 0.001
- added link shaft; visual cylinder length=0.06 radius=0.01
- link base_link: geometry visual cylinder length=0.06 radius=0.04
Joints:
- removed joint base_to_right_leg
- added joint base_link_to_shaft: type continuous, parent base_link, child shaft, origin xyz=0 0 0 rpy=0 0 0, axis 1 0 0
- added joint shaft_joint: type fixed, parent shaft, child propeller, origin xyz=0.0 0 0.02 rpy=0 0 0

Commit message: urdf edits

File: ros_ws/src/motor_p/urdf/motor.urdf (robot description, URDF)
Before this commit: robot motor_urdf, 3 links, 2 joints
Links:
- link shaft: geometry collision cylinder length=0.01 radius=0.06; visual cylinder length=0.06 radius=0.01
