Commit message: Update motor.xacro

File: ros_ws/src/motor_p/urdf/motor.xacro (robot description, xacro)
@@ -16,4 +16,13 @@
       <robotBaseFrame>base_link</robotBaseFrame>
     </plugin>
+  </gazebo>
+  <gazebo reference="base_link">
+    <material>Gazebo/Yellow</material>
+  </gazebo>
+  <gazebo reference="propeller">
+    <material>Gazebo/Turquoise </material>
+  </gazebo>
+  <gazebo reference="shaft">
+    <material>Gazebo/Green</material>
   </gazebo>
   <link name="world"/>

Commit message: added comments.

File: ros_ws/src/motor_p/urdf/motor.xacro (robot description, xacro)
@@ -1,4 +1,6 @@
 <?xml version="1.0"?>
+<!-- The urdf for the motor -->
 <robot name="motor_urdf" xmlns:xacro="http://ros.org/wiki/xacro">
+  <!-- Gazebo plugin diff_drive -->
   <gazebo>
     <plugin name="differential_drive_controller" filename="libgazebo_ros_diff_drive.so">
@@ -17,4 +19,5 @@
     </plugin>
   </gazebo>
+  <!-- Gazebo colors. -->
   <gazebo reference="base_link">
     <material>Gazebo/Yellow</material>
@@ -26,9 +29,11 @@
     <material>Gazebo/Green</material>
   </gazebo>
-  <link name="world"/>
+  <!-- World link to keep motor in place. -->
+  <link name="world" />
   <joint name="fixed" type="fixed">
-    <parent link="world"/>
-    <child link="base_link"/>
+    <parent link="world" />
+    <child link="base_link" />
   </joint>
+  <!--Base link -->
   <link name="base_link">
     <visual>
@@ -50,4 +55,5 @@
     </inertial>
   </link>
+  <!-- Shaft link -->
   <link name="shaft">
     <visual>
@@ -56,4 +62,5 @@
         <cylinder length="0.06" radius="0.01" />
       </geometry>
+      <!-- Colors for RVIZ -->
       <material name="Cyan1">
         <color rgba="0 0.9 0.9 1.0" />
@@ -72,4 +79,5 @@
     </inertial>
   </link>
+  <!-- Propeller link -->
   <link name="propeller">
     <visual>
@@ -78,4 +86,5 @@
         <box size="0.05 0.02 0.001" />
       </geometry>
+      <!-- Colors for RVIZ -->
       <material name="Yellow1">
         <color rgba="0.8 0.8 0 1.0" />
@@ -94,4 +103,5 @@
     </inertial>
   </link>
+  <!-- Shaft joint -->
   <joint name="shaft_joint" type="fixed">
     <origin rpy="0 0 0" xyz="0.0 0 0.02" />
@@ -99,4 +109,5 @@
     <child link="propeller" />
   </joint>
+  <!-- Base link to shaft -->
   <joint name="base_link_to_shaft" type="continuous">
     <axis xyz="1 0 0" />
